File: Conector grove 4 pinos universal/kit.kicad_pcb (KiCad board)
At the start: 2 copper layers, 69.2 x 57.2 mm, 30 parts, among them IC1 ARDUINO_UNO, P1 A0, P10 D6, P11 D7, P12 D8, P13 I2C, P14 I2C, P15 I2C, P16 I2C, P17 D11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

Commit message: Seg Set  4 14:45:49 BRT 2017
Parts:
- P1, P10, P11, P12, P13, P14, P15, P16, P17, P18, P19, P2, P3, P4, P5, P6, P7, P8, P9: footprint MY_kicad:molex_2510 -> MyFootprint:Grove 4 pinos
- R3: value 330 -> 10k
- moved P6 3.61 mm to (64.1, 60.3)
- moved P10 3.56 mm to (64.1, 27.3)
- moved P11 3.56 mm to (42.5, 60.3)
- moved P12 3.56 mm to (42.5, 52.1)
- moved P17 3.56 mm to (42.5, 27.3)
- moved P18 3.56 mm to (42.5, 35.6)
- moved P19 3.56 mm to (42.5, 43.8)
- moved P7 3.56 mm to (64.1, 52.1)
- moved P8 3.56 mm to (64.1, 43.8)
- moved P9 3.56 mm to (64.1, 35.6)
- moved P5 3.43 mm to (82.5, 27.2)
- moved P1 3.43 mm to (82.5, 35.6)
- moved P2 3.43 mm to (82.5, 43.8)
- moved P3 3.43 mm to (82.5, 52.1)
- moved P4 3.43 mm to (82.5, 60.3)
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Routing:
- net VCC: track 247.2 -> 204.3 mm
- net ADC4: track 69.3 -> 55.2 mm
- net D7: track 73.7 -> 66.5 mm
- net RXD: track 19.0 -> 16.5 mm
- net Earth: track 25.4 -> 27.4 mm
- net ADC5: track 57.5 -> 56.1 mm
- net D8: track 50.4 -> 49.3 mm
- net D12: track 13.5 -> 12.9 mm
Other:
- board text added: "TX RX"
- board text removed: "RX TX"
